File: PCB/umami-blade.brd (EAGLE design)
At the start: 260 x 120 mm, 22 parts, among them U1 MCP3008

Commit message: progress
Parts:
- added BATT: 2-pin, RA, SMT, con-jst:S2B-PH-SM4-
- added C2: 0.1uF, rlc:0603-CAP
- added GND, RX, TX: PADSMD-050X050, con-testpoints:SMD-050X050
- added M1: (no value), circuit-monkey-chips:0128A
- added M2, M3: Class-D, 16W, circuit-monkey-chips:0123A
- added MOD1: (no value), display-lcd-oled:PIMORONI-LCD-CONTROLLER
- added PI1: Pi 2W, co-raspberrypi:PI-ZERO-2W
- C1: value (none) -> 0.1uF
- moved C1 255.5 mm to (-32.0, -9.00)
- moved GPIO1 238.5 mm to (-37.0, -17.0)
- moved U1 238.5 mm to (-26.0, -18.0)
- moved TRIGR 156.5 mm to (120.0, 50.0)
- moved TRIGZR 156.5 mm to (110.0, 50.0)
- moved START 151.8 mm to (93.0, -60.0), turned to 90 degrees
- moved A 151.2 mm to (116.0, 20.0), turned to 90 degrees
- moved B 151.2 mm to (106.0, 10.0), turned to 90 degrees
- moved JOY2 151.2 mm to (106.0, -20.0), turned to 180 degrees
- moved X 151.2 mm to (106.0, 30.0), turned to 90 degrees
- moved Y 151.2 mm to (96.0, 20.0), turned to 90 degrees
- moved CAP 148.4 mm to (-93.0, -60.0), turned to 90 degrees
- moved LCD1 146.7 mm to (-1.50, 0.00)
- moved PLUS 145.0 mm to (93.0, 60.0), turned to 90 degrees
- moved DOWN 144.1 mm to (-106.0, -30.0), turned to 90 degrees
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Connections:
- removed net N$2: JOY2.3
- new net !BTN_CS: GPIO1.18, PI1.24
- new net !BTN_IRQ: GPIO1.22, PI1.22
- new net !JOY_CS: PI1.26, U1.10
- new net +4.1V: BATT.1
- new net +5V: M1.5V, MOD1.5V, PI1.2, PI1.4
- new net N$7: JOY2.3, U1.6
- new net RX: PI1.10, RX.1
- new net SPI_CLK: GPIO1.19, PI1.23, U1.13
- new net SPI_DI: GPIO1.24, PI1.19, U1.11
- new net SPI_DO: GPIO1.20, PI1.21, U1.12
- new net TX: PI1.8, TX.1
- net +3.3V: now also C2.1, PI1.1, U1.15, U1.16
- net GND: now also BATT.2, C2.2, GND.1, M1.GNDI, M1.GNDO, M2.GND, M2.GND2, M3.GND, M3.GND2, MOD1.GND@I2S, MOD1.GND@MENU, PI1.14, PI1.20, PI1.25, PI1.30, PI1.34, PI1.39, PI1.6, PI1.9, U1.14, U1.9
- net N$1: now also U1.2
- net N$4: now also U1.3; no longer U1.2
- net N$5: now also U1.5; no longer U1.3
- net N$6: now also U1.7; no longer U1.4
Other:
- board size 260 x 120 mm -> 240 x 132 mm
