File: PCB/umami-blade.sch (EAGLE design)
At the start: 22 parts, among them U1 MCP3008

Commit message: progress
Parts:
- added BATT: 2-pin, RA, SMT, con-jst:02PRA-SMT
- added C2: 0.1uF, rlc:CAPACITOR0603
- added GND, RX, TX: PADSMD-050X050, con-testpoints:PADSMD-050X050
- added M1: (no value), circuit-monkey-chips:0128REV-A
- added M2, M3: Class-D, 16W, circuit-monkey-chips:0123REV-A
- added MOD1: (no value), display-lcd-oled:LCD_CONTROLLERPIMORONI-8IN
- added PI1: Pi 2W, co-raspberrypi:RASPBERRY_PI-ZERO-2W
- C1: value (none) -> 0.1uF
Connections:
- removed net N$2: JOY2.BTN
- new net !BTN_CS: GPIO1.!CS, PI1.24
- new net !BTN_IRQ: GPIO1.!IRQ, PI1.22
- new net !JOY_CS: PI1.26, U1.!CS
- new net +4.1V: BATT.1
- new net +5V: M1.+5, MOD1.5V, PI1.2, PI1.4
- new net N$7: JOY2.BTN, U1.CH5
- new net RX: PI1.10, RX.PAD
- new net SPI_CLK: GPIO1.SCL, PI1.23, U1.CLK
- new net SPI_DI: GPIO1.SI, PI1.19, U1.DIN
- new net SPI_DO: GPIO1.SO, PI1.21, U1.DOUT
- new net TX: PI1.8, TX.PAD
- net +3.3V: now also C2.1, PI1.1, U1.VDD, U1.VREF
- net GND: now also BATT.2, C2.2, GND.PAD, M1.GND, M2.GND, M3.GND, MOD1.GND, PI1.14, PI1.20, PI1.25, PI1.30, PI1.34, PI1.39, PI1.6, PI1.9, U1.AGND, U1.VSS
- net N$1: now also U1.CH1
- net N$4: now also U1.CH2; no longer U1.CH1
- net N$5: now also U1.CH4; no longer U1.CH2
- net N$6: now also U1.CH6; no longer U1.CH3
Other:
- note added: "TODO: - LCD Buttons - Accelerometer - Rumbles - LEDs (neopixel?) - Charger - PWR ON/Off"
- note removed: "TODO: - Raspi - LCD Controller - LCD Buttons - JoyCon w/ FPC"
- moved on the sheet: A, B, C1, CAP, DOWN, GPIO1, JOY1, JOY2, LCD1, LEFT, NEG, PLUS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
